File: board/leds.sch (KiCad schematic (older format))
At the start: 78 parts

Commit message: schematic changes for apa102-2020-6 footprint
Parts:
- D1, D10, D11, D12, D13, D14, D15, D16, D17, D18, D19, D2, D20, D21, D22, D23, D24, D25, D26, D27, D28, D29, D3, D30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: footprint LED_SMD:LED-APA102-2020_tightened_pads -> LED_SMD:LED-APA102-2020-6
