File: board/earthvenusmars.sch (KiCad schematic (older format))
At the start: 27 parts, among them J1 Conn_01x05_Female, J2 Conn_01x02_Female, J4 Conn_01x04, SW1 SW_SPST, SW2 SW_SPST, SW3 SW_SPST, U1 ATSAMD21G18A-AU, U2 MIC5504-3.3YM5, Y1 32768Hz

Commit message: change USB pin connector to 5-pin to handle the ID pin from usb-micro
Parts:
- J4: value Conn_01x04 -> Conn_01x05; footprint Connector_PinHeader_1.27mm:PinHeader_1x04_P1.27mm_Vertical -> Connector_PinHeader_1.27mm:PinHeader_1x05_P1.27mm_Vertical; symbol Connector_Generic:Conn_01x04 -> Connector_Generic:Conn_01x05
Connections:
- net USB_D+: now also J4.3 (Pin_3); no longer J4.2 (Pin_2)
- net USB_D-: now also J4.4 (Pin_4); no longer J4.3 (Pin_3)
- net VBUS: now also J4.5 (Pin_5); no longer J4.4 (Pin_4)
- no-connect marks 23 -> 24
Changed lines of the file:
@@
 L power:GND #PWR0102
 U 1 1 5EB2B290
-P 3750 4550
-F 0 "#PWR0102" H 3750 4300 50  0001 C CNN
-F 1 "GND" V 3755 4422 50  0000 R CNN
-F 2 "" H 3750 4550 50  0001 C CNN
-F 3 "" H 3750 4550 50  0001 C CNN
-	1    3750 4550
+P 3800 4550
+F 0 "#PWR0102" H 3800 4300 50  0001 C CNN
+F 1 "GND" V 3805 4422 50  0000 R CNN
+F 2 "" H 3800 4550 50  0001 C CNN
+F 3 "" H 3800 4550 50  0001 C CNN
+	1    3800 4550
 	-1   0    0    1
 $EndComp
@@
 L power:VBUS #PWR0103
 U 1 1 5EB2B320
-P 3450 4550
-F 0 "#PWR0103" H 3450 4400 50  0001 C CNN
-F 1 "VBUS" V 3465 4677 50  0000 L CNN
-F 2 "" H 3450 4550 50  0001 C CNN
-F 3 "" H 3450 4550 50  0001 C CNN
-	1    3450 4550
+P 3400 4550
+F 0 "#PWR0103" H 3400 4400 50  0001 C CNN
+F 1 "VBUS" V 3415 4677 50  0000 L CNN
+F 2 "" H 3400 4550 50  0001 C CNN
+F 3 "" H 3400 4550 50  0001 C CNN
+	1    3400 4550
 	1    0    0    -1
 $EndComp
@@
 	5400 1750 5500 1750
 $Comp
-L Connector_Generic:Conn_01x04 J4
+L Connector_Generic:Conn_01x05 J4
 U 1 1 5F9E60C8
-P 3650 4750
-F 0 "J4" V 3614 4462 50  0000 R CNN
-F 1 "Conn_01x04" V 3750 4950 50  0000 R CNN
-F 2 "Connector_PinHeader_1.27mm:PinHeader_1x04_P1.27mm_Vertical" H 3650 4750 50  0001 C CNN
-F 3 "~" H 3650 4750 50  0001 C CNN
-	1    3650 4750
+P 3600 4750
+F 0 "J4" V 3564 4462 50  0000 R CNN
+F 1 "Conn_01x05" V 3700 4950 50  0000 R CNN
+F 2 "Connector_PinHeader_1.27mm:PinHeader_1x05_P1.27mm_Vertical" H 3600 4750 50  0001 C CNN
+F 3 "~" H 3600 4750 50  0001 C CNN
+	1    3600 4750
 	0    1    1    0
 $EndComp
@@
 Connection ~ 5350 1550
 Wire Wire Line
-	3950 4150 3650 4150
-Wire Wire Line
-	3650 4150 3650 4550
-Wire Wire Line
-	3950 4050 3550 4050
-Wire Wire Line
-	3550 4050 3550 4550
-Wire Wire Line
 	3950 3950 3650 3950
 Wire Wire Line
@@
 	0    -1   -1   0
 $EndComp
+Wire Wire Line
+	3500 4550 3500 4050
+Wire Wire Line
+	3500 4050 3950 4050
+Wire Wire Line
+	3600 4550 3600 4150
+Wire Wire Line
+	3600 4150 3950 4150
+NoConn ~ 3700 4550
 $EndSCHEMATC

Commit message: rearrange F.Fab and B.Fab layers for clarity to aid assembly engineers; use the larger 0603 footprint for ferrite bead because it's way more manageable and I have the parts
Parts:
- FB1: footprint Inductor_SMD:L_0201_0603Metric -> Inductor_SMD:L_0603_1608Metric
Changed lines of the file:
@@
 F 0 "FB1" H 6250 1096 50  0000 L CNN
 F 1 "220Ω @ 100MHz" H 6250 1005 50  0000 L CNN
-F 2 "Inductor_SMD:L_0201_0603Metric" V 6080 1050 50  0001 C CNN
+F 2 "Inductor_SMD:L_0603_1608Metric" V 6080 1050 50  0001 C CNN
 F 3 "~" H 6150 1050 50  0001 C CNN
 F 4 "BLM03HB191SN1D" H 6150 1050 50  0001 C CNN "Designation"

Commit message: correct part number for new ferrite bead
Parts:
- FB1: Designation BLM03HB191SN1D -> BLM18AG221SN1D
Changed lines of the file:
@@
 F 2 "Inductor_SMD:L_0603_1608Metric" V 6080 1050 50  0001 C CNN
 F 3 "~" H 6150 1050 50  0001 C CNN
-F 4 "BLM03HB191SN1D" H 6150 1050 50  0001 C CNN "Designation"
+F 4 "BLM18AG221SN1D" H 6150 1050 50  0001 C CNN "Designation"
 	1    6150 1050
 	1    0    0    -1
