File: programmer/programmer.kicad_pcb (KiCad board)
At the start: 2 copper layers, 62.2 x 54 mm, 5 parts, among them J1 v1 programmer, J2 v2 programmer, SW1 SW_SPST

Commit message: tiny polish tweaks
Parts:
- renumbered SW1 to RESET
Changed lines of the file:
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@@
     (thickness 1.6)
     (drawings 25)
-    (tracks 64)
+    (tracks 71)
     (zones 0)
     (modules 5)
@@
       (effects (font (size 0.8 0.8) (thickness 0.1)))
     )
-    (fp_text user 3.3V (at -4.496 -1.7782 270) (layer F.SilkS)
+    (fp_text user 3.3V (at -4.496 -1.7782 -90 unlocked) (layer F.SilkS)
       (effects (font (size 0.6 0.6) (thickness 0.08)))
     )
@@
     (descr "Ultraminiature Surface Mount Slide Switch, right-angle, https://www.ckswitches.com/media/1424/pcm.pdf")
     (attr smd)
-    (fp_text reference SW1 (at -0.126132 -4.434126 112) (layer F.SilkS)
+    (fp_text reference RESET (at 1.614433 -3.511087 112) (layer F.SilkS)
       (effects (font (size 1 1) (thickness 0.15)))
     )
@@
   (gr_circle (center 115.4 93.2) (end 115.512 93.2) (layer F.SilkS) (width 0.4))
   (gr_circle (center 96 89.7) (end 96.2106 89.7) (layer F.SilkS) (width 0.4))
-  (gr_circle (center 95.2 106.4) (end 95.4 106.4) (layer F.SilkS) (width 0.4))
+  (gr_circle (center 96.9 107.4) (end 97.1 107.4) (layer F.SilkS) (width 0.4))
   (gr_circle (center 100 100) (end 116.856113 100) (layer F.SilkS) (width 0.12))
   (gr_circle (center 100 100) (end 111.059976 100) (layer F.SilkS) (width 0.12))
@@
   (segment (start 100 100) (end 100 99.2) (width 0.25) (layer B.Cu) (net 3))
   (segment (start 103.033604 102.4) (end 104 102.4) (width 0.25) (layer F.Cu) (net 4))
-  (segment (start 101.27 100.636396) (end 103.033604 102.4) (width 0.25) (layer F.Cu) (net 4))
-  (segment (start 101.27 100) (end 101.27 100.636396) (width 0.25) (layer F.Cu) (net 4))
   (via (at 101.97316 102.36984) (size 0.8) (drill 0.4) (layers F.Cu B.Cu) (net 4))
   (segment (start 103.033604 102.4) (end 102.00332 102.4) (width 0.25) (layer F.Cu) (net 4))
@@
   (segment (start 101.219 103.124) (end 101.346 102.997) (width 0.25) (layer B.Cu) (net 4))
   (segment (start 80.4164 104.1146) (end 82.7532 103.1494) (width 0.25) (layer B.Cu) (net 4))
-  (via (at 80.4164 104.1146) (size 0.8) (drill 0.4) (layers F.Cu B.Cu) (net 4))
   (segment (start 79.502 107.442) (end 78.746628 109.2781) (width 0.25) (layer F.Cu) (net 4))
-  (segment (start 80.4164 104.1146) (end 79.502 107.442) (width 0.25) (layer F.Cu) (net 4))
   (segment (start 112.071966 110.471966) (end 104 102.4) (width 0.25) (layer F.Cu) (net 4))
   (segment (start 126.049536 110.775491) (end 112.071966 110.471966) (width 0.25) (layer F.Cu) (net 4))
+  (segment (start 101.27 100.636396) (end 101.97316 102.36984) (width 0.25) (layer F.Cu) (net 4))
+  (segment (start 101.27 100) (end 101.27 100.636396) (width 0.25) (layer F.Cu) (net 4))
+  (via (at 79.5 106.8) (size 0.8) (drill 0.4) (layers F.Cu B.Cu) (net 4))
+  (segment (start 79.502 106.802) (end 79.5 106.8) (width 0.25) (layer F.Cu) (net 4))
+  (segment (start 79.502 107.442) (end 79.502 106.802) (width 0.25) (layer F.Cu) (net 4))
+  (segment (start 79.5 105.031) (end 80.4164 104.1146) (width 0.25) (layer B.Cu) (net 4))
+  (segment (start 79.5 106.8) (end 79.5 105.031) (width 0.25) (layer B.Cu) (net 4))
   (segment (start 103.314001 104.114001) (end 102.9 103.7) (width 0.25) (layer B.Cu) (net 5))
   (segment (start 102.9 100.36) (end 102.9 103.7) (width 0.25) (layer B.Cu) (net 5))
   (segment (start 102.54 100) (end 102.9 100.36) (width 0.25) (layer B.Cu) (net 5))
-  (segment (start 82.99 103.7) (end 102.9 103.7) (width 0.25) (layer B.Cu) (net 5))
-  (segment (start 79.0956 105.8418) (end 82.99 103.7) (width 0.25) (layer B.Cu) (net 5))
-  (via (at 79.0956 105.8418) (size 0.8) (drill 0.4) (layers F.Cu B.Cu) (net 5))
-  (segment (start 77.622808 106.496549) (end 79.0956 105.8418) (width 0.25) (layer F.Cu) (net 5))
   (segment (start 129.719984 111.95814) (end 129.868841 111.809283) (width 0.25) (layer F.Cu) (net 5))
   (segment (start 129.784702 112.315015) (end 129.61114 111.95814) (width 0.25) (layer F.Cu) (net 5))
@@
   (segment (start 129.1082 113.9444) (end 129.784702 112.315015) (width 0.25) (layer B.Cu) (net 5))
   (segment (start 128.816783 114.663362) (end 129.1082 113.9444) (width 0.25) (layer B.Cu) (net 5))
+  (via (at 81 104.7) (size 0.8) (drill 0.4) (layers F.Cu B.Cu) (net 5))
+  (segment (start 82.99 103.7) (end 102.9 103.7) (width 0.25) (layer B.Cu) (net 5))
+  (segment (start 81.6 104.4) (end 82.99 103.7) (width 0.25) (layer B.Cu) (net 5))
+  (segment (start 81.42 104.5) (end 81.6 104.4) (width 0.25) (layer B.Cu) (net 5))
+  (segment (start 81 104.7) (end 81.42 104.5) (width 0.25) (layer B.Cu) (net 5))
+  (segment (start 79.0956 105.8044) (end 77.622808 106.496549) (width 0.25) (layer F.Cu) (net 5))
+  (segment (start 79.9 105.3) (end 79.0956 105.8044) (width 0.25) (layer F.Cu) (net 5))
+  (segment (start 81 104.7) (end 79.9 105.3) (width 0.25) (layer F.Cu) (net 5))
 )
